File: power.kicad_sch (KiCad schematic)
At the start: 18 parts, among them U4 TPS61040DBV, U5 TPS7A2050PDBV

Commit message: overhausl inputs a lot
read too much, thought too much.
try one with the "just 0R plus a nice big good quality cap" from the TI
precision seminar, describing common realities, as well as mixing in
what they did on the ads1262ref scale design document for the second
channel with a more "full blown" input filter.

I don't really like how none of this seems to be a proper AA filter,
but... ok.
Parts:
- C11, C6, C7: symbol karl-marel-atomics:KC0805_22uF_25V -> karl-atomic-basic:KC0805_22uF_25V
- C12: symbol karl-marel-atomics:KC0603_33pF -> karl-atomic-basic:KC0603_33pF
- C13, C14: symbol karl-marel-atomics:KC0805_10uF_25V -> karl-atomic-basic:KC0805_10uF_25V
- C8: symbol karl-marel-atomics:KC0603_1uF -> karl-atomic-basic:KC0603_1uF
- R5: symbol karl-marel-atomics:KR0603_100k -> karl-atomic-basic:KR0603_100k
- R6: symbol karl-marel-atomics:KR0603_360k -> karl-atomic-basic:KR0603_360k
- R7: symbol karl-marel-atomics:KR0603_1R -> karl-atomic-basic:KR0603_1R
Changed lines of the file:
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@@
 	)
 	(symbol
-		(lib_id "karl-marel-atomics:KR0603_360k")
+		(lib_id "karl-atomic-basic:KR0603_360k")
 		(at 127 58.42 0)
 		(unit 1)
@@
 	)
 	(symbol
-		(lib_id "karl-marel-atomics:KC0805_10uF_25V")
+		(lib_id "karl-atomic-basic:KC0805_10uF_25V")
 		(at 149.86 106.68 0)
 		(unit 1)
@@
 	)
 	(symbol
-		(lib_id "karl-marel-atomics:KC0805_22uF_25V")
+		(lib_id "karl-atomic-basic:KC0805_22uF_25V")
 		(at 81.28 60.96 0)
 		(unit 1)
@@
 	)
 	(symbol
-		(lib_id "karl-marel-atomics:KC0805_22uF_25V")
+		(lib_id "karl-atomic-basic:KC0805_22uF_25V")
 		(at 93.98 106.68 0)
 		(unit 1)
@@
 	)
 	(symbol
-		(lib_id "karl-marel-atomics:KC0603_1uF")
+		(lib_id "karl-atomic-basic:KC0603_1uF")
 		(at 139.7 106.68 0)
 		(unit 1)
@@
 	)
 	(symbol
-		(lib_id "karl-marel-atomics:KR0603_1R")
+		(lib_id "karl-atomic-basic:KR0603_1R")
 		(at 86.36 101.6 90)
 		(unit 1)
@@
 	)
 	(symbol
-		(lib_id "karl-marel-atomics:KR0603_100k")
+		(lib_id "karl-atomic-basic:KR0603_100k")
 		(at 127 68.58 0)
 		(unit 1)
@@
 	)
 	(symbol
-		(lib_id "karl-marel-atomics:KC0805_22uF_25V")
+		(lib_id "karl-atomic-basic:KC0805_22uF_25V")
 		(at 104.14 106.68 0)
 		(unit 1)
@@
 	)
 	(symbol
-		(lib_id "karl-marel-atomics:KC0805_10uF_25V")
+		(lib_id "karl-atomic-basic:KC0805_10uF_25V")
 		(at 147.32 63.5 0)
 		(unit 1)
@@
 	)
 	(symbol
-		(lib_id "karl-marel-atomics:KC0603_33pF")
+		(lib_id "karl-atomic-basic:KC0603_33pF")
 		(at 137.16 58.42 0)
 		(unit 1)

Commit message: moarh updates
we commit to save our progress
Parts:
- JP3: footprint Jumper:SolderJumper-2_P1.3mm_Open_TrianglePad1.0x1.5mm -> jlc-extras:SolderJumper-2_P1.3mm_Open_TrianglePad0.9x1.8mm
Changed lines of the file:
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@@
 			)
 		)
-		(property "Footprint" "Jumper:SolderJumper-2_P1.3mm_Open_TrianglePad1.0x1.5mm"
+		(property "Footprint" "jlc-extras:SolderJumper-2_P1.3mm_Open_TrianglePad0.9x1.8mm"
 			(at 113.03 165.1 0)
 			(effects
